File: KiCAD/uad/uab_logic.sch (KiCad schematic (older format))
At the start: 10 parts

Commit message: разведена плата кнопок, плата контроллера - не расставлены светодиоды
Parts:
- added HL3, HL4, HL5, HL6, HL7, HL8, HL9: Светодиод, N_VD_HL:Светодиод_SMD_0603, symbol elements:Светодиод
- added R12, R13: 300 Ом(0805), N_RLC:Резистор_SMD_0805_0,125Вт, symbol elements:Резистор_0,125Вт
- added R14, R15, R16, R17, R18, R19, R20: 100 Ом(0805), N_RLC:Резистор_SMD_0805_0,125Вт, symbol elements:Резистор_0,125Вт
- added VD1: Диод_шоттки, N_VD_HL:Диод_BAR43CFILM_SOT-23, symbol MOTOR:Диод_шоттки
- added VT1, VT2: PBSS4540Z, N_VD_HL:Транзистор_NPN_SOT223, symbol elements:Транзистор_NPN_1Б-2(4)К-3Э_0
- added XP6: Вилка_PLD6_ПРОГ, N_X:Вилка_PLD6_вертикальная, symbol elements:Вилка_PLD6_ПРОГ
- added XS1, XS2, XS3, XS4, XS5: Розетка_PBS3, N_X:Розетка_PBS3_вертикальная, symbol elements:Розетка_PBS3
Connections:
- net labels added: BUT_8_IN, LED_1, LED_2, LED_3, LED_4, LED_5, LED_6, LED_7, LED_8, PWR_GND
- net labels removed: BUT_0_IN, LED_work
- wire segments 60 -> 105
- no-connect marks 3 -> 4

Commit message: начато добавление клеммников на схему
Parts:
- added C? (x2): 4.7мкФ(1210), N_RLC:Конденсатор_SMD_1210, symbol elements:Конденсатор_керамический
- added FU? (x2): Предохранитель, symbol elements:Предохранитель
- added X?: L_220, symbol elements:отверстие_под_пайку
- added X?: N_220, symbol elements:отверстие_под_пайку
- added XТ? (x3): Клеммник_х2, N_X:Клеммник_х2_шаг5, symbol elements:Клеммник_х2
Connections:
- net labels added: PWR_12V
- wire segments 105 -> 127
Other:
- note added: "Вход 220В"
- note added: "На 1\nвентилятор\n"
- note added: "На 2\nвентилятор\n"

Commit message: не поставлен эмиттерный повторитель на питание логики
Parts:
- added C?: 4.7мкФ(1210), N_RLC:Конденсатор_SMD_1210, symbol elements:Конденсатор_керамический
- added FU?: Предохранитель, N_RLC:Предохранитель_R700, symbol elements:Предохранитель
- added VD? (x4): Шоттки_BAR43CFILM, N_VD_HL:Диод_BAR43CFILM_SOT-23, symbol MOTOR:Диод_шоттки
- added X?: L_12, N_X:ОтверстиеD1.2, symbol elements:отверстие_под_пайку
- added X?: N_12, N_X:ОтверстиеD1.2, symbol elements:отверстие_под_пайку
- FU1, FU2: renamed from FU?; footprint (none) -> N_RLC:Предохранитель_R700
- VD1: value Диод_шоттки -> Шоттки_BAR43CFILM
- X1, X2: renamed from X?; footprint (none) -> N_X:ОтверстиеD1.2
- gave numbers to parts that had none: 5
Connections:
- wire segments 127 -> 156

Commit message: обе схемы закончены, разводка второй платы не закончена
Parts:
- removed FU2: Предохранитель, N_RLC:Предохранитель_R700, symbol elements:Предохранитель
- removed VD? (x4): Шоттки_BAR43CFILM, N_VD_HL:Диод_BAR43CFILM_SOT-23, symbol MOTOR:Диод_шоттки
- added G1: Стабилиатор_LM2931AZ-5.0G, N_G:Стабилизатор_корпус_TO-92, symbol elements:стабилизатор_нерегулируемый_LM2931
- added L1, L2, L3: 33мкГн, N_RLC:Чип-индуктивность_SMD_0805, symbol elements:Чип-индуктивность
- added VD2: Мост_DB155S, N_VD_HL:Диод_матрица_корпус_DB-1S, symbol elements:Диодный_мост(DB-1S)
- added VD3: Шоттки_BAR43CFILM, N_VD_HL:Диод_BAR43CFILM_SOT-23, symbol MOTOR:Диод_шоттки
- FU1: footprint N_RLC:Предохранитель_R700 -> N_RLC:Предохранитель_MF-R_d10.4
- FU2: renamed from FU?; footprint N_RLC:Предохранитель_R700 -> N_RLC:Предохранитель_MF-R_d10.4
- XT1, XT2, XT3: footprint N_X:Клеммник_х2_шаг5 -> N_X:Клеммник_х2_шаг2.54
- gave numbers to parts that had none: 3
Connections:
- net labels added: L1, L1_12, L2, L2_12, N1, N1_12
- net labels removed: D_Out_1, D_Out_2, D_Out_3, D_Out_4, D_Out_5, D_Out_6, D_Out_7, D_Out_8
- wire segments 156 -> 152

Commit message: закончена разводка первого варианта (без отскока) и без фрезеровки
Parts:
- removed VD1, VD3: Шоттки_BAR43CFILM, N_VD_HL:Диод_BAR43CFILM_SOT-23, symbol MOTOR:Диод_шоттки
- added VD1, VD3: Шоттки_BAR43CFILM, N_VD_HL:Диод_BAR43CFILM_SOT-23, symbol elements:Диод_шоттки
- added XP7: Вилка_PLS3, N_X:Вилка_PLS3_вертикальная, symbol elements:Вилка_PLS3
Connections:
- net labels added: collector_1, collector_2
- wire segments 152 -> 155
Changed lines of the file:
@@
 BUT_COM_OUT
 Text Label 2125 8500 0    50   ~ 0
-GND
+VCC
 Text Label 2125 8400 0    50   ~ 0
 GND
@@
 GND
 Text Label 2125 9100 0    50   ~ 0
-GND
+VCC
 Text Label 4375 9700 0    50   ~ 0
 BUT_1_IN
@@
 Text Label 7825 2875 0    50   ~ 0
 TX
+Text Label 5050 2775 2    50   ~ 0
+PWM_OUT_1
+Wire Wire Line
+	5050 2675 5400 2675
 Text Label 5050 2675 2    50   ~ 0
-PWM_OUT_1
-Wire Wire Line
-	5050 2675 5400 2675
-Text Label 5050 2775 2    50   ~ 0
 PWM_OUT_2
 Wire Wire Line
@@
 Text Label 12700 2325 0    50   ~ 0
 GND
-$Comp
-L MOTOR:Диод_шоттки VD1
-U 1 1 5C2E11EB
-P 12700 2025
-F 0 "VD1" H 12900 2150 50  0000 C CNN
-F 1 "Шоттки_BAR43CFILM" H 13275 1950 50  0000 C CNN
-F 2 "N_VD_HL:Диод_BAR43CFILM_SOT-23" H 12600 2025 50  0001 C CNN
-F 3 "" H 12600 2025 50  0001 C CNN
-	1    12700 2025
-	1    0    0    -1
-$EndComp
 Wire Wire Line
 	13000 2025 13250 2025
@@
 Вход 220В
 Text Notes 4725 4450 0    50   ~ 0
+На 2\nвентилятор\n
+Text Notes 4725 5100 0    50   ~ 0
 На 1\nвентилятор\n
-Text Notes 4725 5100 0    50   ~ 0
-На 2\nвентилятор\n
 $Comp
 L elements:отверстие_под_пайку X3
@@
 Text Label 14775 8675 0    50   ~ 0
 VCC
-$Comp
-L MOTOR:Диод_шоттки VD3
-U 1 1 5C44939A
-P 14300 8675
-F 0 "VD3" H 14500 8800 50  0000 C CNN
-F 1 "Шоттки_BAR43CFILM" H 14875 8600 50  0000 C CNN
-F 2 "N_VD_HL:Диод_BAR43CFILM_SOT-23" H 14200 8675 50  0001 C CNN
-F 3 "" H 14200 8675 50  0001 C CNN
-	1    14300 8675
-	1    0    0    -1
-$EndComp
 Wire Wire Line
 	14600 8675 14775 8675
@@
 Wire Wire Line
 	11550 9175 10525 9175
+Text Label 6400 4500 0    50   ~ 0
+collector_2
+Text Label 6400 5150 0    50   ~ 0
+collector_1
+$Comp
+L elements:Диод_шоттки VD1
+U 1 1 5C2E30A1
+P 12700 2025
+F 0 "VD1" H 12850 2200 50  0000 C CNN
+F 1 "Шоттки_BAR43CFILM" H 13325 1925 50  0000 C CNN
+F 2 "N_VD_HL:Диод_BAR43CFILM_SOT-23" H 12600 2025 50  0001 C CNN
+F 3 "" H 12600 2025 50  0001 C CNN
+	1    12700 2025
+	1    0    0    -1
+$EndComp
+$Comp
+L elements:Диод_шоттки VD3
+U 1 1 5C2F4AB9
+P 14300 8675
+F 0 "VD3" H 14450 8850 50  0000 C CNN
+F 1 "Шоттки_BAR43CFILM" H 14925 8575 50  0000 C CNN
+F 2 "N_VD_HL:Диод_BAR43CFILM_SOT-23" H 14200 8675 50  0001 C CNN
+F 3 "" H 14200 8675 50  0001 C CNN
+	1    14300 8675
+	1    0    0    -1
+$EndComp
+$Comp
+L elements:Вилка_PLS3 XP7
+U 1 1 5C2D9B36
+P 1325 7475
+F 0 "XP7" H 1581 7556 60  0000 C CNN
+F 1 "Вилка_PLS3" H 1525 6900 60  0001 C CNN
+F 2 "N_X:Вилка_PLS3_вертикальная" H 1325 7475 60  0001 C CNN
+F 3 "" H 1325 7475 60  0001 C CNN
+	1    1325 7475
+	1    0    0    -1
+$EndComp
+Wire Wire Line
+	1825 7575 2125 7575
+Text Label 2125 7575 0    50   ~ 0
+GND
+Wire Wire Line
+	1825 7675 2125 7675
+Wire Wire Line
+	1825 7775 2125 7775
+Text Label 2125 7675 0    50   ~ 0
+RX
+Text Label 2125 7775 0    50   ~ 0
+TX
 $EndSCHEMATC
