File: KiCAD/uad/uad_sensor.sch (KiCad schematic (older format))
At the start: 21 parts

Commit message: разведена плата кнопок, плата контроллера - не расставлены светодиоды
Changed lines of the file:
@@
 	6375 3825 6300 3825
 Wire Wire Line
-	1300 4800 1600 4800
+	1300 4600 1600 4600
 Wire Wire Line
 	1300 4700 1600 4700
@@
 	1300 5300 1600 5300
 Wire Wire Line
+	1300 5400 1600 5400
+Wire Wire Line
+	1300 4800 1600 4800
+Wire Wire Line
 	1300 5200 1600 5200
 Wire Wire Line
-	1300 4600 1600 4600
-Wire Wire Line
-	1300 5400 1600 5400
+	3550 4700 3850 4700
 Wire Wire Line
 	3550 4800 3850 4800
 Wire Wire Line
-	3550 4700 3850 4700
+	3550 5400 3850 5400
+Wire Wire Line
+	3550 4600 3850 4600
+Wire Wire Line
+	3550 5900 3850 5900
 Wire Wire Line
 	3550 5300 3850 5300
@@
 	3550 5200 3850 5200
 Wire Wire Line
-	3550 4600 3850 4600
-Wire Wire Line
-	3550 5400 3850 5400
-Wire Wire Line
 	3550 5800 3850 5800
-Wire Wire Line
-	3550 5900 3850 5900
 Text Label 1775 1850 0    50   ~ 0
 BUT_COM_OUT
@@
 Text Label 6375 3825 0    50   ~ 0
 GND
-Text Label 1600 4600 0    50   ~ 0
+Text Label 1600 4800 0    50   ~ 0
 BUT_COM_OUT
-Text Label 1600 5400 0    50   ~ 0
+Text Label 1600 5200 0    50   ~ 0
 BUT_COM_OUT
 Text Label 1600 4700 0    50   ~ 0
 GND
-Text Label 1600 4800 0    50   ~ 0
+Text Label 1600 4600 0    50   ~ 0
 GND
-Text Label 1600 5200 0    50   ~ 0
+Text Label 1600 5400 0    50   ~ 0
 GND
 Text Label 1600 5300 0    50   ~ 0
 GND
+Text Label 3850 5900 0    50   ~ 0
+BUT_1_IN
+Text Label 3850 4800 0    50   ~ 0
+BUT_2_IN
+Text Label 3850 4700 0    50   ~ 0
+BUT_3_IN
 Text Label 3850 4600 0    50   ~ 0
-BUT_1_IN
-Text Label 3850 4700 0    50   ~ 0
-BUT_2_IN
-Text Label 3850 4800 0    50   ~ 0
-BUT_3_IN
+BUT_4_IN
+Text Label 3850 5400 0    50   ~ 0
+BUT_5_IN
+Text Label 3850 5300 0    50   ~ 0
+BUT_6_IN
 Text Label 3850 5200 0    50   ~ 0
-BUT_4_IN
-Text Label 3850 5300 0    50   ~ 0
-BUT_5_IN
-Text Label 3850 5400 0    50   ~ 0
-BUT_6_IN
+BUT_7_IN
 Text Label 3850 5800 0    50   ~ 0
-BUT_7_IN
-Text Label 3850 5900 0    50   ~ 0
 BUT_8_IN
 $Comp

Commit message: закончена разводка первого варианта (без отскока) и без фрезеровки
Connections:
- net labels added: VCC_1, VCC_2
Changed lines of the file:
@@
 BUT_COM_OUT
 Text Label 1600 4700 0    50   ~ 0
-GND
+VCC_1
 Text Label 1600 4600 0    50   ~ 0
 GND
@@
 GND
 Text Label 1600 5300 0    50   ~ 0
-GND
+VCC_2
 Text Label 3850 5900 0    50   ~ 0
 BUT_1_IN
