File: KiCAD/uad/uad_analog_panel.sch (KiCad schematic (older format))
At the start: 4 parts

Commit message: добавлены STEP и GERBER файлы
Parts:
- added C16, C17, C18, C19, C20, C21, C22, C23, C24: 100пФ(0603), N_RLC:Конденсатор_SMD_0603, symbol elements:Конденсатор_керамический
- added HL10, HL11, HL12, HL13, HL14, HL15, HL16, HL17, HL18: Светодиод_NeoPixel, N_VD_HL:Светодиод_SMD_neopixel_ws2812b, symbol elements:Светодиод_NeoPixel
- added XP12, XP13, XP14, XP15, XP16, XP17: Вилка_PLS3, N_X:Вилка_PLS3_угловая_вертикальная, symbol elements:Вилка_PLS3
Connections:
- wire segments 6 -> 135
